Commit message: Update aruco marker origin links for isaacsim

File: drop_container_description/urdf/drop_container.urdf (robot description, URDF)
Before this commit: robot drop_container, 17 links, 16 joints
Links:
- link aruco_01_1: geometry collision box size=0.001 0.03 0.03; visual box size=0.001 0.03 0.03
- link aruco_02_1: geometry collision box size=0.001 0.03 0.03; visual box size=0.001 0.03 0.03
- link aruco_03_1: geometry collision box size=0.001 0.03 0.03; visual box size=0.001 0.03 0.03
- link aruco_04_1: geometry collision box size=0.001 0.03 0.03; visual box size=0.001 0.03 0.03
- link aruco_05_1: geometry collision box size=0.001 0.03 0.03; visual box size=0.001 0.03 0.03
- link aruco_06_1: geometry collision box size=0.001 0.03 0.03; visual box size=0.001 0.03 0.03
- link aruco_07_1: geometry collision box size=0.001 0.03 0.03; visual box size=0.001 0.03 0.03
- link aruco_08_1: geometry collision box size=0.001 0.03 0.03; visual box size=0.001 0.03 0.03
- link aruco_09_1: geometry collision box size=0.001 0.03 0.03; visual box size=0.001 0.03 0.03
- link aruco_10_1: geometry collision box size=0.001 0.03 0.03; visual box size=0.001 0.03 0.03
- link aruco_11_1: geometry collision box size=0.001 0.03 0.03; visual box size=0.001 0.03 0.03
- link aruco_12_1: geometry collision box size=0.001 0.03 0.03; visual box size=0.001 0.03 0.03
- link aruco_13_1: geometry collision box size=0.001 0.03 0.03; visual box size=0.001 0.03 0.03
- link aruco_14_1: geometry collision box size=0.001 0.03 0.03; visual box size=0.001 0.03 0.03
- link aruco_15_1: geometry collision box size=0.001 0.03 0.03; visual box size=0.001 0.03 0.03
Joints:
- joint Rigid 1: origin xyz=-0.0875 0.0 -0.0025 rpy=0 0 0 -> xyz=0.0 -0.116 0.1435 rpy=1.5708 0 0
- joint Rigid 10: origin xyz=-0.0875 0.0 -0.0025 rpy=0 0 0 -> xyz=0.0 0.058 0.1435 rpy=1.5708 0 0
- joint Rigid 11: origin xyz=-0.0875 0.0 -0.0025 rpy=0 0 0 -> xyz=0.0 0.058 0.0855 rpy=1.5708 0 0
- joint Rigid 12: origin xyz=-0.0875 0.0 -0.0025 rpy=0 0 0 -> xyz=0.0 0.058 0.0295 rpy=1.5708 0 0
- joint Rigid 13: origin xyz=-0.0875 0.0 -0.0025 rpy=0 0 0 -> xyz=0.0 0.116 0.1435 rpy=1.5708 0 0
- joint Rigid 14: origin xyz=-0.0875 0.0 -0.0025 rpy=0 0 0 -> xyz=0.0 0.116 0.0855 rpy=1.5708 0 0
- joint Rigid 15: origin xyz=-0.0875 0.0 -0.0025 rpy=0 0 0 -> xyz=0.0 0.116 0.0295 rpy=1.5708 0 0
- joint Rigid 2: origin xyz=-0.0875 0.0 -0.0025 rpy=0 0 0 -> xyz=0.0 -0.116 0.0855 rpy=1.5708 0 0
- joint Rigid 3: origin xyz=-0.0875 0.0 -0.0025 rpy=0 0 0 -> xyz=0.0 -0.116 0.0295 rpy=1.5708 0 0
- joint Rigid 4: origin xyz=-0.0875 0.0 -0.0025 rpy=0 0 0 -> xyz=0.0 -0.058 0.1435 rpy=1.5708 0 0
- joint Rigid 5: origin xyz=-0.0875 0.0 -0.0025 rpy=0 0 0 -> xyz=0.0 -0.058 0.0855 rpy=1.5708 0 0
- joint Rigid 6: origin xyz=-0.0875 0.0 -0.0025 rpy=0 0 0 -> xyz=0.0 -0.058 0.0295 rpy=1.5708 0 0
- joint Rigid 7: origin xyz=-0.0875 0.0 -0.0025 rpy=0 0 0 -> xyz=0.0 0.0 0.1435 rpy=1.5708 0 0
- joint Rigid 8: origin xyz=-0.0025 0.0 0.0875 rpy=0 0 0 -> xyz=0.0 0.0 0.0855 rpy=0 0 0
- joint Rigid 9: origin xyz=-0.0875 0.0 -0.0025 rpy=0 0 0 -> xyz=0.0 0.0 0.0295 rpy=1.5708 0 0

File: drop_container_description/urdf/drop_container.xacro (robot description, xacro)
@@ -44,304 +44,320 @@
   </collision>
 </link>
+<!-- ArUco Marker 1: Row 1, Col 1 (Top-Left) -->
 <link name="aruco_01_1">
   <inertial>
-    <origin xyz="0.08549999999999998 -0.1105000000000001 0.14800000000000008" rpy="0 0 0"/>
-    <mass value="0.007065000000000037"/>
-    <inertia ixx="1e-06" iyy="1e-06" izz="1e-06" ixy="0.0" iyz="-0.0" ixz="0.0"/>
-  </inertial>
-  <visual>
-    <origin xyz="0.175 0.0 -0.0535" rpy="0 0 0"/>
-    <geometry>
-      <mesh filename="file://$(find drop_container_description)/meshes/aruco_01_1.stl" scale="0.001 0.001 0.001"/>
-    </geometry>
-    <material name="silver"/>
-  </visual>
-  <collision>
-    <origin xyz="0.175 0.0 -0.0535" rpy="0 0 0"/>
-    <geometry>
-      <mesh filename="file://$(find drop_container_description)/meshes/aruco_01_1.stl" scale="0.001 0.001 0.001"/>
-    </geometry>
-  </collision>
-</link>
+    <origin xyz="0 0 0" rpy="0 0 0"/>
+    <mass value="0.007065000000000037"/>
+    <inertia ixx="1e-06" iyy="1e-06" izz="1e-06" ixy="0.0" iyz="0.0" ixz="0.0"/>
+  </inertial>
+  <visual>
+    <origin xyz="0 0 0" rpy="0 0 0"/>
+    <geometry>
+      <box size="0.001 0.03 0.03"/>
+    </geometry>
+    <material name="silver"/>
+  </visual>
+  <collision>
+    <origin xyz="0 0 0" rpy="0 0 0"/>
+    <geometry>
+      <box size="0.001 0.03 0.03"/>
+    </geometry>
+  </collision>
+</link>
+<!-- ArUco Marker 2: Row 2, Col 1 -->
 <link name="aruco_02_1">
   <inertial>
-    <origin xyz="0.08549999999999996 -0.11050000000000008 0.09" rpy="0 0 0"/>
-    <mass value="0.007065000000000037"/>
-    <inertia ixx="1e-06" iyy="1e-06" izz="1e-06" ixy="-0.0" iyz="-0.0" ixz="-0.0"/>
-  </inertial>
-  <visual>
-    <origin xyz="0.175 0.0 -0.0535" rpy="0 0 0"/>
-    <geometry>
-      <mesh filename="file://$(find drop_container_description)/meshes/aruco_02_1.stl" scale="0.001 0.001 0.001"/>
-    </geometry>
-    <material name="silver"/>
-  </visual>
-  <collision>
-    <origin xyz="0.175 0.0 -0.0535" rpy="0 0 0"/>
-    <geometry>
-      <mesh filename="file://$(find drop_container_description)/meshes/aruco_02_1.stl" scale="0.001 0.001 0.001"/>
-    </geometry>
-  </collision>
-</link>
+    <origin xyz="0 0 0" rpy="0 0 0"/>
+    <mass value="0.007065000000000037"/>
+    <inertia ixx="1e-06" iyy="1e-06" izz="1e-06" ixy="0.0" iyz="0.0" ixz="0.0"/>
+  </inertial>
+  <visual>
+    <origin xyz="0 0 0" rpy="0 0 0"/>
+    <geometry>
+      <box size="0.001 0.03 0.03"/>
+    </geometry>
+    <material name="silver"/>
+  </visual>
+  <collision>
+    <origin xyz="0 0 0" rpy="0 0 0"/>
+    <geometry>
+      <box size="0.001 0.03 0.03"/>
+    </geometry>
+  </collision>
+</link>
+<!-- ArUco Marker 3: Row 3, Col 1 (Bottom-Left) -->
 <link name="aruco_03_1">
   <inertial>
-    <origin xyz="0.08549999999999998 -0.11050000000000006 0.031999999999999994" rpy="0 0 0"/>
-    <mass value="0.007065000000000037"/>
-    <inertia ixx="1e-06" iyy="1e-06" izz="1e-06" ixy="0.0" iyz="0.0" ixz="-0.0"/>
-  </inertial>
-  <visual>
-    <origin xyz="0.175 0.0 -0.0535" rpy="0 0 0"/>
-    <geometry>
-      <mesh filename="file://$(find drop_container_description)/meshes/aruco_03_1.stl" scale="0.001 0.001 0.001"/>
-    </geometry>
-    <material name="silver"/>
-  </visual>
-  <collision>
-    <origin xyz="0.175 0.0 -0.0535" rpy="0 0 0"/>
-    <geometry>
-      <mesh filename="file://$(find drop_container_description)/meshes/aruco_03_1.stl" scale="0.001 0.001 0.001"/>
-    </geometry>
-  </collision>
-</link>
+    <origin xyz="0 0 0" rpy="0 0 0"/>
+    <mass value="0.007065000000000037"/>
+    <inertia ixx="1e-06" iyy="1e-06" izz="1e-06" ixy="0.0" iyz="0.0" ixz="0.0"/>
+  </inertial>
+  <visual>
+    <origin xyz="0 0 0" rpy="0 0 0"/>
+    <geometry>
+      <box size="0.001 0.03 0.03"/>
+    </geometry>
+    <material name="silver"/>
+  </visual>
+  <collision>
+    <origin xyz="0 0 0" rpy="0 0 0"/>
+    <geometry>
+      <box size="0.001 0.03 0.03"/>
+    </geometry>
+  </collision>
+</link>
+<!-- ArUco Marker 4: Row 1, Col 2 -->
 <link name="aruco_04_1">
   <inertial>
-    <origin xyz="0.08549999999999998 -0.05525000000000008 0.14800000000000008" rpy="0 0 0"/>
-    <mass value="0.007065000000000037"/>
-    <inertia ixx="1e-06" iyy="1e-06" izz="1e-06" ixy="0.0" iyz="0.0" ixz="-0.0"/>
-  </inertial>
-  <visual>
-    <origin xyz="0.175 0.0 -0.0535" rpy="0 0 0"/>
-    <geometry>
-      <mesh filename="file://$(find drop_container_description)/meshes/aruco_04_1.stl" scale="0.001 0.001 0.001"/>
-    </geometry>
-    <material name="silver"/>
-  </visual>
-  <collision>
-    <origin xyz="0.175 0.0 -0.0535" rpy="0 0 0"/>
-    <geometry>
-      <mesh filename="file://$(find drop_container_description)/meshes/aruco_04_1.stl" scale="0.001 0.001 0.001"/>
-    </geometry>
-  </collision>
-</link>
+    <origin xyz="0 0 0" rpy="0 0 0"/>
+    <mass value="0.007065000000000037"/>
+    <inertia ixx="1e-06" iyy="1e-06" izz="1e-06" ixy="0.0" iyz="0.0" ixz="0.0"/>
+  </inertial>
+  <visual>
+    <origin xyz="0 0 0" rpy="0 0 0"/>
+    <geometry>
+      <box size="0.001 0.03 0.03"/>
+    </geometry>
+    <material name="silver"/>
+  </visual>
+  <collision>
+    <origin xyz="0 0 0" rpy="0 0 0"/>
+    <geometry>
+      <box size="0.001 0.03 0.03"/>
+    </geometry>
+  </collision>
+</link>
+<!-- ArUco Marker 5: Row 2, Col 2 -->
 <link name="aruco_05_1">
   <inertial>
-    <origin xyz="0.08549999999999998 -0.05525000000000006 0.09000000000000005" rpy="0 0 0"/>
-    <mass value="0.007065000000000037"/>
-    <inertia ixx="1e-06" iyy="1e-06" izz="1e-06" ixy="-0.0" iyz="0.0" ixz="-0.0"/>
-  </inertial>
-  <visual>
-    <origin xyz="0.175 0.0 -0.0535" rpy="0 0 0"/>
-    <geometry>
-      <mesh filename="file://$(find drop_container_description)/meshes/aruco_05_1.stl" scale="0.001 0.001 0.001"/>
-    </geometry>
-    <material name="silver"/>
-  </visual>
-  <collision>
-    <origin xyz="0.175 0.0 -0.0535" rpy="0 0 0"/>
-    <geometry>
-      <mesh filename="file://$(find drop_container_description)/meshes/aruco_05_1.stl" scale="0.001 0.001 0.001"/>
-    </geometry>
-  </collision>
-</link>
+    <origin xyz="0 0 0" rpy="0 0 0"/>
+    <mass value="0.007065000000000037"/>
+    <inertia ixx="1e-06" iyy="1e-06" izz="1e-06" ixy="0.0" iyz="0.0" ixz="0.0"/>
+  </inertial>
+  <visual>
+    <origin xyz="0 0 0" rpy="0 0 0"/>
+    <geometry>
+      <box size="0.001 0.03 0.03"/>
+    </geometry>
+    <material name="silver"/>
+  </visual>
+  <collision>
+    <origin xyz="0 0 0" rpy="0 0 0"/>
+    <geometry>
+      <box size="0.001 0.03 0.03"/>
+    </geometry>
+  </collision>
+</link>
+<!-- ArUco Marker 6: Row 3, Col 2 -->
 <link name="aruco_06_1">
   <inertial>
-    <origin xyz="0.08549999999999998 -0.05525000000000006 0.03200000000000002" rpy="0 0 0"/>
-    <mass value="0.007065000000000037"/>
-    <inertia ixx="1e-06" iyy="1e-06" izz="1e-06" ixy="0.0" iyz="0.0" ixz="0.0"/>
-  </inertial>
-  <visual>
-    <origin xyz="0.175 0.0 -0.0535" rpy="0 0 0"/>
-    <geometry>
-      <mesh filename="file://$(find drop_container_description)/meshes/aruco_06_1.stl" scale="0.001 0.001 0.001"/>
-    </geometry>
-    <material name="silver"/>
-  </visual>
-  <collision>
-    <origin xyz="0.175 0.0 -0.0535" rpy="0 0 0"/>
-    <geometry>
-      <mesh filename="file://$(find drop_container_description)/meshes/aruco_06_1.stl" scale="0.001 0.001 0.001"/>
-    </geometry>
-  </collision>
-</link>
+    <origin xyz="0 0 0" rpy="0 0 0"/>
+    <mass value="0.007065000000000037"/>
+    <inertia ixx="1e-06" iyy="1e-06" izz="1e-06" ixy="0.0" iyz="0.0" ixz="0.0"/>
+  </inertial>
+  <visual>
+    <origin xyz="0 0 0" rpy="0 0 0"/>
+    <geometry>
+      <box size="0.001 0.03 0.03"/>
+    </geometry>
+    <material name="silver"/>
+  </visual>
+  <collision>
+    <origin xyz="0 0 0" rpy="0 0 0"/>
+    <geometry>
+      <box size="0.001 0.03 0.03"/>
+    </geometry>
+  </collision>
+</link>
+<!-- ArUco Marker 7: Row 1, Col 3 -->
 <link name="aruco_07_1">
   <inertial>
-    <origin xyz="0.08550000000000002 -8.829151401759714e-17 0.14800000000000008" rpy="0 0 0"/>
-    <mass value="0.007065000000000037"/>
-    <inertia ixx="1e-06" iyy="1e-06" izz="1e-06" ixy="0.0" iyz="0.0" ixz="0.0"/>
-  </inertial>
-  <visual>
-    <origin xyz="0.175 0.0 -0.0535" rpy="0 0 0"/>
-    <geometry>
-      <mesh filename="file://$(find drop_container_description)/meshes/aruco_07_1.stl" scale="0.001 0.001 0.001"/>
-    </geometry>
-    <material name="silver"/>
-  </visual>
-  <collision>
-    <origin xyz="0.175 0.0 -0.0535" rpy="0 0 0"/>
-    <geometry>
-      <mesh filename="file://$(find drop_container_description)/meshes/aruco_07_1.stl" scale="0.001 0.001 0.001"/>
-    </geometry>
-  </collision>
-</link>
+    <origin xyz="0 0 0" rpy="0 0 0"/>
+    <mass value="0.007065000000000037"/>
+    <inertia ixx="1e-06" iyy="1e-06" izz="1e-06" ixy="0.0" iyz="0.0" ixz="0.0"/>
+  </inertial>
+  <visual>
+    <origin xyz="0 0 0" rpy="0 0 0"/>
+    <geometry>
+      <box size="0.001 0.03 0.03"/>
+    </geometry>
+    <material name="silver"/>
+  </visual>
+  <collision>
+    <origin xyz="0 0 0" rpy="0 0 0"/>
+    <geometry>
+      <box size="0.001 0.03 0.03"/>
+    </geometry>
+  </collision>
+</link>
+<!-- ArUco Marker 8: Row 2, Col 3 (CENTER) -->
 <link name="aruco_08_1">
   <inertial>
-    <origin xyz="0.0004999999999999866 -7.302800339756536e-17 5.551115123125783e-17" rpy="0 0 0"/>
-    <mass value="0.007065000000000037"/>
-    <inertia ixx="1e-06" iyy="1e-06" izz="1e-06" ixy="0.0" iyz="-0.0" ixz="-0.0"/>
-  </inertial>
-  <visual>
-    <origin xyz="0.09 0.0 -0.1435" rpy="0 0 0"/>
-    <geometry>
-      <mesh filename="file://$(find drop_container_description)/meshes/aruco_08_1.stl" scale="0.001 0.001 0.001"/>
-    </geometry>
-    <material name="silver"/>
-  </visual>
-  <collision>
-    <origin xyz="0.09 0.0 -0.1435" rpy="0 0 0"/>
-    <geometry>
-      <mesh filename="file://$(find drop_container_description)/meshes/aruco_08_1.stl" scale="0.001 0.001 0.001"/>
-    </geometry>
-  </collision>
-</link>
+    <origin xyz="0 0 0" rpy="0 0 0"/>
+    <mass value="0.007065000000000037"/>
+    <inertia ixx="1e-06" iyy="1e-06" izz="1e-06" ixy="0.0" iyz="0.0" ixz="0.0"/>
+  </inertial>
+  <visual>
+    <origin xyz="0 0 0" rpy="0 0 0"/>
+    <geometry>
+      <box size="0.001 0.03 0.03"/>
+    </geometry>
+    <material name="silver"/>
+  </visual>
+  <collision>
+    <origin xyz="0 0 0" rpy="0 0 0"/>
+    <geometry>
+      <box size="0.001 0.03 0.03"/>
+    </geometry>
+  </collision>
+</link>
+<!-- ArUco Marker 9: Row 3, Col 3 -->
 <link name="aruco_09_1">
   <inertial>
-    <origin xyz="0.08549999999999996 -5.825792523292263e-17 0.03200000000000002" rpy="0 0 0"/>
-    <mass value="0.007065000000000037"/>
-    <inertia ixx="1e-06" iyy="1e-06" izz="1e-06" ixy="-0.0" iyz="-0.0" ixz="0.0"/>
-  </inertial>
-  <visual>
-    <origin xyz="0.175 0.0 -0.0535" rpy="0 0 0"/>
-    <geometry>
-      <mesh filename="file://$(find drop_container_description)/meshes/aruco_09_1.stl" scale="0.001 0.001 0.001"/>
-    </geometry>
-    <material name="silver"/>
-  </visual>
-  <collision>
-    <origin xyz="0.175 0.0 -0.0535" rpy="0 0 0"/>
-    <geometry>
-      <mesh filename="file://$(find drop_container_description)/meshes/aruco_09_1.stl" scale="0.001 0.001 0.001"/>
-    </geometry>
-  </collision>
-</link>
+    <origin xyz="0 0 0" rpy="0 0 0"/>
+    <mass value="0.007065000000000037"/>
+    <inertia ixx="1e-06" iyy="1e-06" izz="1e-06" ixy="0.0" iyz="0.0" ixz="0.0"/>
+  </inertial>
+  <visual>
+    <origin xyz="0 0 0" rpy="0 0 0"/>
+    <geometry>
+      <box size="0.001 0.03 0.03"/>
+    </geometry>
+    <material name="silver"/>
+  </visual>
+  <collision>
+    <origin xyz="0 0 0" rpy="0 0 0"/>
+    <geometry>
+      <box size="0.001 0.03 0.03"/>
+    </geometry>
+  </collision>
+</link>
+<!-- ArUco Marker 10: Row 1, Col 4 -->
 <link name="aruco_10_1">
   <inertial>
-    <origin xyz="0.08549999999999998 0.05524999999999992 0.14800000000000008" rpy="0 0 0"/>
-    <mass value="0.007065000000000037"/>
-    <inertia ixx="1e-06" iyy="1e-06" izz="1e-06" ixy="0.0" iyz="0.0" ixz="0.0"/>
-  </inertial>
-  <visual>
-    <origin xyz="0.175 0.0 -0.0535" rpy="0 0 0"/>
-    <geometry>
-      <mesh filename="file://$(find drop_container_description)/meshes/aruco_10_1.stl" scale="0.001 0.001 0.001"/>
-    </geometry>
-    <material name="silver"/>
-  </visual>
-  <collision>
-    <origin xyz="0.175 0.0 -0.0535" rpy="0 0 0"/>
-    <geometry>
-      <mesh filename="file://$(find drop_container_description)/meshes/aruco_10_1.stl" scale="0.001 0.001 0.001"/>
-    </geometry>
-  </collision>
-</link>
+    <origin xyz="0 0 0" rpy="0 0 0"/>
+    <mass value="0.007065000000000037"/>
+    <inertia ixx="1e-06" iyy="1e-06" izz="1e-06" ixy="0.0" iyz="0.0" ixz="0.0"/>
+  </inertial>
+  <visual>
+    <origin xyz="0 0 0" rpy="0 0 0"/>
+    <geometry>
+      <box size="0.001 0.03 0.03"/>
+    </geometry>
+    <material name="silver"/>
+  </visual>
+  <collision>
+    <origin xyz="0 0 0" rpy="0 0 0"/>
+    <geometry>
+      <box size="0.001 0.03 0.03"/>
+    </geometry>
+  </collision>
+</link>
+<!-- ArUco Marker 11: Row 2, Col 4 -->
 <link name="aruco_11_1">
   <inertial>
-    <origin xyz="0.08549999999999996 0.055249999999999924 0.09000000000000005" rpy="0 0 0"/>
-    <mass value="0.007065000000000037"/>
-    <inertia ixx="1e-06" iyy="1e-06" izz="1e-06" ixy="0.0" iyz="-0.0" ixz="-0.0"/>
-  </inertial>
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