Commit message: Update gripper center offset

File: JETANK_description/urdf/JETANK.xacro (robot description, xacro)
@@ -532,5 +532,5 @@
 </joint>
 <joint name="GRIPPER_CENTER" type="fixed">
-  <origin xyz="-0.095065 0 0" rpy="0 0 0"/>
+  <origin xyz="-0.108750 0 0" rpy="0 0 0"/>
   <parent link="GRIPPER_BASE_1"/>
   <child link="GRIPPER_CENTER_LINK"/>

Commit message: Add material colors

File: JETANK_description/urdf/JETANK.xacro (robot description, xacro)
@@ -15,5 +15,5 @@
       <mesh filename="file://$(find JETANK_description)/meshes/base_link.stl" scale="0.001 0.001 0.001"/>
     </geometry>
-    <material name="silver"/>
+    <material name="base_link_material"/>
   </visual>
   <collision>
@@ -35,5 +35,5 @@
       <mesh filename="file://$(find JETANK_description)/meshes/ANTENNA_L_1.stl" scale="0.001 0.001 0.001"/>
     </geometry>
-    <material name="silver"/>
+    <material name="antenna_material"/>
   </visual>
   <collision>
@@ -55,5 +55,5 @@
       <mesh filename="file://$(find JETANK_description)/meshes/BEARING_1.stl" scale="0.001 0.001 0.001"/>
     </geometry>
-    <material name="silver"/>
+    <material name="bearing_material"/>
   </visual>
   <collision>
@@ -75,5 +75,5 @@
       <mesh filename="file://$(find JETANK_description)/meshes/ARM_LOWER_1.stl" scale="0.001 0.001 0.001"/>
     </geometry>
-    <material name="silver"/>
+    <material name="arm_material"/>
   </visual>
   <collision>
@@ -95,5 +95,5 @@
       <mesh filename="file://$(find JETANK_description)/meshes/FREE_WHEEL_L_1.stl" scale="0.001 0.001 0.001"/>
     </geometry>
-    <material name="silver"/>
+    <material name="wheel_material"/>
   </visual>
   <collision>
@@ -115,5 +115,5 @@
       <mesh filename="file://$(find JETANK_description)/meshes/FREE_WHEEL_R_1.stl" scale="0.001 0.001 0.001"/>
     </geometry>
-    <material name="silver"/>
+    <material name="wheel_material"/>
   </visual>
   <collision>
@@ -135,5 +135,5 @@
       <mesh filename="file://$(find JETANK_description)/meshes/CAMERA_1.stl" scale="0.001 0.001 0.001"/>
     </geometry>
-    <material name="silver"/>
+    <material name="camera_material"/>
   </visual>
   <collision>
@@ -155,5 +155,5 @@
       <mesh filename="file://$(find JETANK_description)/meshes/CAM_HOLDER_1.stl" scale="0.001 0.001 0.001"/>
     </geometry>
-    <material name="silver"/>
+    <material name="camera_holder_material"/>
   </visual>
   <collision>
@@ -175,5 +175,5 @@
       <mesh filename="file://$(find JETANK_description)/meshes/GRIPPER_L1_1.stl" scale="0.001 0.001 0.001"/>
     </geometry>
-    <material name="silver"/>
+    <material name="gripper_material"/>
   </visual>
   <collision>
@@ -195,5 +195,5 @@
       <mesh filename="file://$(find JETANK_description)/meshes/GRIPPER_L2_1.stl" scale="0.001 0.001 0.001"/>
     </geometry>
-    <material name="silver"/>
+    <material name="gripper_material"/>
   </visual>
   <collision>
@@ -215,5 +215,5 @@
       <mesh filename="file://$(find JETANK_description)/meshes/SERVO_UPPER_1.stl" scale="0.001 0.001 0.001"/>
     </geometry>
-    <material name="silver"/>
+    <material name="servo_material"/>
   </visual>
   <collision>
@@ -235,5 +235,5 @@
       <mesh filename="file://$(find JETANK_description)/meshes/ARM_MIDDLE_2.stl" scale="0.001 0.001 0.001"/>
     </geometry>
-    <material name="silver"/>
+    <material name="arm_material"/>
   </visual>
   <collision>
@@ -255,5 +255,5 @@
       <mesh filename="file://$(find JETANK_description)/meshes/SERVO_LOWER_1.stl" scale="0.001 0.001 0.001"/>
     </geometry>
-    <material name="silver"/>
+    <material name="servo_material"/>
   </visual>
   <collision>
@@ -275,5 +275,5 @@
       <mesh filename="file://$(find JETANK_description)/meshes/DRIVER_WHEEL_R_2.stl" scale="0.001 0.001 0.001"/>
     </geometry>
-    <material name="silver"/>
+    <material name="wheel_material"/>
   </visual>
   <collision>
@@ -295,5 +295,5 @@
       <mesh filename="file://$(find JETANK_description)/meshes/DRIVER_WHEEL_L_1.stl" scale="0.001 0.001 0.001"/>
     </geometry>
-    <material name="silver"/>
+    <material name="wheel_material"/>
   </visual>
   <collision>
@@ -315,5 +315,5 @@
       <mesh filename="file://$(find JETANK_description)/meshes/GRIPPER_R2_1.stl" scale="0.001 0.001 0.001"/>
     </geometry>
-    <material name="silver"/>
+    <material name="gripper_material"/>
   </visual>
   <collision>
@@ -335,5 +335,5 @@
       <mesh filename="file://$(find JETANK_description)/meshes/GRIPPER_R1_1.stl" scale="0.001 0.001 0.001"/>
     </geometry>
-    <material name="silver"/>
+    <material name="gripper_material"/>
   </visual>
   <collision>
@@ -355,5 +355,5 @@
       <mesh filename="file://$(find JETANK_description)/meshes/GRIPPER_BASE_1.stl" scale="0.001 0.001 0.001"/>
     </geometry>
-    <material name="silver"/>
+    <material name="gripper_material"/>
   </visual>
   <collision>
@@ -375,5 +375,5 @@
       <box size="0.01 0.01 0.01"/>
     </geometry>
-    <material name="silver"/>
+    <material name="gripper_material"/>
   </visual>
   <collision>
@@ -395,5 +395,5 @@
       <mesh filename="file://$(find JETANK_description)/meshes/ARM_UPPER_1.stl" scale="0.001 0.001 0.001"/>
     </geometry>
-    <material name="silver"/>
+    <material name="arm_material"/>
   </visual>
   <collision>
@@ -415,5 +415,5 @@
       <mesh filename="file://$(find JETANK_description)/meshes/ANTENNA_R_2.stl" scale="0.001 0.001 0.001"/>
     </geometry>
-    <material name="silver"/>
+    <material name="antenna_material"/>
   </visual>
   <collision>

File: JETANK_description/urdf/materials.xacro (robot description, xacro)
@@ -1,4 +1,33 @@
 <?xml version="1.0" ?>
 <robot name="JETANK" xmlns:xacro="http://www.ros.org/wiki/xacro" >
+<!-- Base materials from jetank_description -->
+<material name="base_link_material">
+  <color rgba="0.25 0.25 0.25 1"/>
+</material>
+<material name="arm_material">
+  <color rgba="0.41 0.45 0.39 1"/>
+</material>
+<material name="wheel_material">
+  <color rgba="0.5 0.5 0.4 1"/>
+</material>
+<material name="camera_material">
+  <color rgba="0.84 0.74 0.60 1"/>
+</material>
+<material name="camera_holder_material">
+  <color rgba="0.0 0.5 0.5 1"/>
+</material>
+<material name="antenna_material">
+  <color rgba="0.2 0.2 0.2 1"/>
+</material>
+<material name="servo_material">
+  <color rgba="0.58 0.78 0.78 1"/>
+</material>
+<material name="gripper_material">
+  <color rgba="0.65 0.65 0.62 1"/>
+</material>
+<material name="bearing_material">
+  <color rgba="0.67 0.74 0.67 1"/>
+</material>
+<!-- Keep original silver as fallback -->
 <material name="silver">
   <color rgba="0.700 0.700 0.700 1.000"/>

Commit message: Add Ignition Gazebo simulation with camera sensors and YOLOE verification
- Add RGB, depth, and segmentation camera sensors to JETANK.gazebo (Ignition Fortress)
- Add camera_optical_frame link/joint to JETANK.xacro, fix zero-inertia links
- Create lego_world.sdf with table, colored blocks, and lightweight camera model
- Create gazebo.launch.py for headless Ignition Gazebo with ros_gz_bridge
- Add verify_detections.py for comparing YOLOE poses against ground truth
- Update setup.py with worlds data and verify_detections entry point

File: JETANK_description/urdf/JETANK.xacro (robot description, xacro)
@@ -168,5 +168,5 @@
     <origin xyz="-0.01499953892313019 4.862891752669459e-05 0.0029999309597343315" rpy="0 0 0"/>
     <mass value="0.0062442558314246485"/>
-    <inertia ixx="0.0" iyy="1e-06" izz="1e-06" ixy="0.0" iyz="0.0" ixz="0.0"/>
+    <inertia ixx="1e-06" iyy="1e-06" izz="1e-06" ixy="0.0" iyz="0.0" ixz="0.0"/>
   </inertial>
   <visual>
@@ -188,5 +188,5 @@
     <origin xyz="-0.0024363716844204852 0.003974526639710773 0.003008312151974085" rpy="0 0 0"/>
     <mass value="0.02146027585992414"/>
-    <inertia ixx="0.0" iyy="6e-06" izz="6e-06" ixy="-1e-06" iyz="-0.0" ixz="-0.0"/>
+    <inertia ixx="1e-06" iyy="6e-06" izz="6e-06" ixy="-1e-06" iyz="-0.0" ixz="-0.0"/>
   </inertial>
   <visual>
@@ -328,5 +328,5 @@
     <origin xyz="-0.014999865534495699 4.7716893300363966e-05 0.002999957523558139" rpy="0 0 0"/>
     <mass value="0.006244255831424672"/>
-    <inertia ixx="0.0" iyy="1e-06" izz="1e-06" ixy="0.0" iyz="0.0" ixz="0.0"/>
+    <inertia ixx="1e-06" iyy="1e-06" izz="1e-06" ixy="0.0" iyz="0.0" ixz="0.0"/>
   </inertial>
   <visual>
@@ -548,3 +548,16 @@
   <child link="ANTENNA_R_2"/>
 </joint>
+<!-- Camera optical frame (OpenCV convention: X-right, Y-down, Z-forward) -->
+<link name="camera_optical_frame">
+  <inertial>
+    <origin xyz="0 0 0" rpy="0 0 0"/>
+    <mass value="0.001"/>
+    <inertia ixx="1e-06" iyy="1e-06" izz="1e-06" ixy="0" iyz="0" ixz="0"/>
+  </inertial>
+</link>
+<joint name="camera_optical_joint" type="fixed">
+  <origin xyz="0 0 0" rpy="-1.5707963 0 -1.5707963"/>
+  <parent link="CAMERA_1"/>
+  <child link="camera_optical_frame"/>
+</joint>
 </robot>

Commit message: Add Gazebo joint control pipeline and DiffDrive for JETANK simulation
- Add JointPositionController plugins for all 8 arm/gripper joints
  with Gazebo default PID (no custom gains)
- Add DiffDrive plugin for drive wheels with odometry publishing
- Add joint_command_bridge node: splits /joint_commands into per-joint
  Float64 topics that Gazebo JointPositionController plugins listen on
- Update gazebo.launch.py: spawn JETANK via ros_gz_sim create, bridge
  joint command and cmd_vel topics, sequence startup with OnProcessExit
- GUI now publishes to both /joint_states (RViz) and /joint_commands
  (Gazebo), and publishes zero cmd_vel for DiffDrive active braking
- Simplify motion button handlers to use cmd_vel directly
- Add base_footprint link for mobile robot convention
- Change drive wheels to continuous joints for unlimited rotation
- Set wheel friction: all wheels mu=5.0 for ground grip
- Update arm/gripper joint limits to match SC15 servo specs
  (effort 2.0/1.0 N·m, velocity 6.5 rad/s)

File: JETANK_description/urdf/JETANK.xacro (robot description, xacro)
@@ -4,4 +4,11 @@
 <xacro:include filename="$(find JETANK_description)/urdf/JETANK.trans" />
 <xacro:include filename="$(find JETANK_description)/urdf/JETANK.gazebo" />
+<!-- base_footprint: ground projection of the robot (mobile robot convention) -->
+<link name="base_footprint"/>
+<joint name="base_joint" type="fixed">
+  <origin xyz="0 0 0.08" rpy="0 0 0"/>
+  <parent link="base_footprint"/>
+  <child link="base_link"/>
+</joint>
 <link name="base_link">
   <inertial>
@@ -439,5 +446,5 @@
   <child link="ARM_LOWER_1"/>
   <axis xyz="-4e-06 -0.002097 0.999998"/>
-  <limit upper="1.8" lower="-1.8" effort="100" velocity="100"/>
+  <limit upper="1.8" lower="-1.8" effort="2.0" velocity="6.5"/>
 </joint>
 <joint name="revolute_FREE_WHEEL_LEFT" type="revolute">
@@ -465,5 +472,5 @@
   <child link="CAM_HOLDER_1"/>
   <axis xyz="0 1 0"/>
-  <limit upper="1.0" lower="-1.0" effort="100" velocity="100"/>
+  <limit upper="1.0" lower="-1.0" effort="2.0" velocity="6.5"/>
 </joint>
 <joint name="revolute_GRIPPER_L1" type="revolute">
@@ -472,5 +479,5 @@
   <child link="GRIPPER_L1_1"/>
   <axis xyz="-5e-06 -0.002097 0.999998"/>
-  <limit upper="0.0" lower="-1.047198" effort="100" velocity="100"/>
+  <limit upper="0.0" lower="-1.047198" effort="1.0" velocity="6.5"/>
 </joint>
 <joint name="revolute_GRIPPER_L2" type="revolute">
@@ -479,5 +486,5 @@
   <child link="GRIPPER_L2_1"/>
   <axis xyz="5e-06 0.002097 -0.999998"/>
-  <limit upper="0.0" lower="-1.047198" effort="100" velocity="100"/>
+  <limit upper="0.0" lower="-1.047198" effort="1.0" velocity="6.5"/>
 </joint>
 <joint name="Revolute_SERVO_UPPER" type="revolute">
@@ -486,5 +493,5 @@
   <child link="SERVO_UPPER_1"/>
   <axis xyz="-0.003633 -0.999991 -0.002097"/>
-  <limit upper="1.0" lower="-1.548620" effort="100" velocity="100"/>
+  <limit upper="1.0" lower="-1.548620" effort="2.0" velocity="6.5"/>
 </joint>
 <joint name="Revolute_SERVO_LOWER" type="revolute">
@@ -493,5 +500,5 @@
   <child link="ARM_MIDDLE_2"/>
   <axis xyz="-0.003633 -0.999991 -0.002097"/>
-  <limit upper="1.574492" lower="-1.892348" effort="100" velocity="100"/>
+  <limit upper="1.574492" lower="-1.892348" effort="2.0" velocity="6.5"/>
 </joint>
 <joint name="Rigid_SERVO_LOWER_ARM_LOWER" type="fixed">
@@ -500,17 +507,17 @@
   <child link="SERVO_LOWER_1"/>
 </joint>
-<joint name="Revolute_DRIVING_WHEEL_R" type="revolute">
+<joint name="Revolute_DRIVING_WHEEL_R" type="continuous">
   <origin xyz="0.054631 0.033431 -0.052049" rpy="0 0 0"/>
   <parent link="base_link"/>
   <child link="DRIVER_WHEEL_R_2"/>
   <axis xyz="-0.003633 -0.999991 -0.002097"/>
-  <limit upper="6.283185" lower="0.0" effort="100" velocity="100"/>
-</joint>
-<joint name="Revolute_DRIVING_WHEEL_L" type="revolute">
+  <limit effort="100" velocity="100"/>
+</joint>
+<joint name="Revolute_DRIVING_WHEEL_L" type="continuous">
   <origin xyz="-0.064189 -0.054537 -0.052234" rpy="0 0 0"/>
   <parent link="base_link"/>
   <child link="DRIVER_WHEEL_L_1"/>
   <axis xyz="0.003633 0.999991 0.002097"/>
-  <limit upper="6.283185" lower="0.0" effort="100" velocity="100"/>
+  <limit effort="100" velocity="100"/>
 </joint>
 <joint name="Revolute_GRIPPER_R2" type="revolute">
@@ -519,5 +526,5 @@
   <child link="GRIPPER_R2_1"/>
   <axis xyz="-5e-06 -0.002097 0.999998"/>
-  <limit upper="0.0" lower="-1.047198" effort="100" velocity="100"/>
+  <limit upper="0.0" lower="-1.047198" effort="1.0" velocity="6.5"/>
 </joint>
 <joint name="Revolute_GRIPPER_R1" type="revolute">
@@ -526,5 +533,5 @@
   <child link="GRIPPER_R1_1"/>
   <axis xyz="-5e-06 -0.002097 0.999998"/>
-  <limit upper="1.047198" lower="0.0" effort="100" velocity="100"/>
+  <limit upper="1.047198" lower="0.0" effort="1.0" velocity="6.5"/>
 </joint>
 <joint name="rigid_GRIPPER_BASE_ARM_UPPER" type="fixed">

Commit message: Fix Gazebo wheel drift and arm oscillation
Wheels:
- Normalize wheel joint Z origins to equalize ground contact height
- Fix XY origins to mesh hole centers
- Change free wheels from revolute to continuous (no rotation limits)
- Replace wheel collision meshes with cylinder primitives
- Normalize all wheel joint axes to pure Y
- Reduce free wheel friction from 5.0 to 0.1 (caster behavior)
- Add light damping (0.01) to free wheel joints

Arm:
- Add tuned PID gains to all 8 arm JointPositionController plugins
- Add passive damping to all 8 arm revolute joints

World physics:
- Increase ODE solver iterations to 200 with SOR 1.3
- Add contact_surface_layer for stable wheel-ground contact
- Add friction and min_depth to ground plane collision

Reduces idle drift from ~0.5mm/s to ~0.17mm/s.

File: JETANK_description/urdf/JETANK.xacro (robot description, xacro)
@@ -105,7 +105,7 @@
   </visual>
   <collision>
-    <origin xyz="-0.05431 0.054968 0.052234" rpy="0 0 0"/>
-    <geometry>
-      <mesh filename="file://$(find JETANK_description)/meshes/FREE_WHEEL_L_1.stl" scale="0.001 0.001 0.001"/>
+    <origin xyz="0 -0.01353 0" rpy="1.5707963 0 0"/>
+    <geometry>
+      <cylinder radius="0.02486" length="0.04476"/>
     </geometry>
   </collision>
@@ -125,7 +125,7 @@
   </visual>
   <collision>
-    <origin xyz="0.063868 -0.033862 0.052048" rpy="0 0 0"/>
-    <geometry>
-      <mesh filename="file://$(find JETANK_description)/meshes/FREE_WHEEL_R_1.stl" scale="0.001 0.001 0.001"/>
+    <origin xyz="0 0.01353 0" rpy="1.5707963 0 0"/>
+    <geometry>
+      <cylinder radius="0.02486" length="0.04476"/>
     </geometry>
   </collision>
@@ -285,7 +285,7 @@
   </visual>
   <collision>
-    <origin xyz="-0.054631 -0.033431 0.052049" rpy="0 0 0"/>
-    <geometry>
-      <mesh filename="file://$(find JETANK_description)/meshes/DRIVER_WHEEL_R_2.stl" scale="0.001 0.001 0.001"/>
+    <origin xyz="0 0.01902 0" rpy="1.5707963 0 0"/>
+    <geometry>
+      <cylinder radius="0.02734" length="0.03903"/>
     </geometry>
   </collision>
@@ -305,7 +305,7 @@
   </visual>
   <collision>
-    <origin xyz="0.064189 0.054537 0.052234" rpy="0 0 0"/>
-    <geometry>
-      <mesh filename="file://$(find JETANK_description)/meshes/DRIVER_WHEEL_L_1.stl" scale="0.001 0.001 0.001"/>
+    <origin xyz="0 -0.01902 0" rpy="1.5707963 0 0"/>
+    <geometry>
+      <cylinder radius="0.02734" length="0.03903"/>
     </geometry>
   </collision>
@@ -447,18 +447,19 @@
   <axis xyz="-4e-06 -0.002097 0.999998"/>
   <limit upper="1.8" lower="-1.8" effort="2.0" velocity="6.5"/>
-</joint>
-<joint name="revolute_FREE_WHEEL_LEFT" type="revolute">
-  <origin xyz="0.05431 -0.054968 -0.052234" rpy="0 0 0"/>
+  <dynamics damping="0.5"/>
+</joint>
+<joint name="revolute_FREE_WHEEL_LEFT" type="continuous">
+  <origin xyz="0.054304 -0.054100 -0.053366" rpy="0 0 0"/>
   <parent link="base_link"/>
   <child link="FREE_WHEEL_L_1"/>
-  <axis xyz="0.003633 0.999991 0.002097"/>
-  <limit upper="6.283185" lower="0.0" effort="100" velocity="100"/>
-</joint>
-<joint name="revolute_FREE_WHEEL_RIGHT" type="revolute">
-  <origin xyz="-0.063868 0.033862 -0.052048" rpy="0 0 0"/>
+  <axis xyz="0 1 0"/>
+  <dynamics damping="0.01"/>
+</joint>
+<joint name="revolute_FREE_WHEEL_RIGHT" type="continuous">
+  <origin xyz="-0.063847 0.033000 -0.053410" rpy="0 0 0"/>
   <parent link="base_link"/>
   <child link="FREE_WHEEL_R_1"/>
-  <axis xyz="-0.003633 -0.999991 -0.002097"/>
-  <limit upper="6.283185" lower="0.0" effort="100" velocity="100"/>
+  <axis xyz="0 -1 0"/>
+  <dynamics damping="0.01"/>
 </joint>
 <joint name="rigid_CAMERA_CAMERA_HOLDER" type="fixed">
@@ -473,4 +474,5 @@
   <axis xyz="0 1 0"/>
   <limit upper="1.0" lower="-1.0" effort="2.0" velocity="6.5"/>
+  <dynamics damping="0.2"/>
 </joint>
 <joint name="revolute_GRIPPER_L1" type="revolute">
@@ -480,4 +482,5 @@
   <axis xyz="-5e-06 -0.002097 0.999998"/>
   <limit upper="0.0" lower="-1.047198" effort="1.0" velocity="6.5"/>
+  <dynamics damping="0.1"/>
 </joint>
 <joint name="revolute_GRIPPER_L2" type="revolute">
@@ -487,4 +490,5 @@
   <axis xyz="5e-06 0.002097 -0.999998"/>
   <limit upper="0.0" lower="-1.047198" effort="1.0" velocity="6.5"/>
+  <dynamics damping="0.1"/>
 </joint>
 <joint name="Revolute_SERVO_UPPER" type="revolute">
@@ -494,4 +498,5 @@
   <axis xyz="-0.003633 -0.999991 -0.002097"/>
   <limit upper="1.0" lower="-1.548620" effort="2.0" velocity="6.5"/>
+  <dynamics damping="0.3"/>
 </joint>
 <joint name="Revolute_SERVO_LOWER" type="revolute">
@@ -501,4 +506,5 @@
   <axis xyz="-0.003633 -0.999991 -0.002097"/>
   <limit upper="1.574492" lower="-1.892348" effort="2.0" velocity="6.5"/>
+  <dynamics damping="0.3"/>
 </joint>
 <joint name="Rigid_SERVO_LOWER_ARM_LOWER" type="fixed">
@@ -508,15 +514,15 @@
 </joint>
 <joint name="Revolute_DRIVING_WHEEL_R" type="continuous">
-  <origin xyz="0.054631 0.033431 -0.052049" rpy="0 0 0"/>
+  <origin xyz="0.054634 0.032570 -0.050948" rpy="0 0 0"/>
   <parent link="base_link"/>
   <child link="DRIVER_WHEEL_R_2"/>
-  <axis xyz="-0.003633 -0.999991 -0.002097"/>
+  <axis xyz="0 -1 0"/>
   <limit effort="100" velocity="100"/>
 </joint>
 <joint name="Revolute_DRIVING_WHEEL_L" type="continuous">
-  <origin xyz="-0.064189 -0.054537 -0.052234" rpy="0 0 0"/>
+  <origin xyz="-0.064218 -0.053670 -0.050868" rpy="0 0 0"/>
   <parent link="base_link"/>
   <child link="DRIVER_WHEEL_L_1"/>
-  <axis xyz="0.003633 0.999991 0.002097"/>
+  <axis xyz="0 1 0"/>
   <limit effort="100" velocity="100"/>
 </joint>
@@ -527,4 +533,5 @@
   <axis xyz="-5e-06 -0.002097 0.999998"/>
   <limit upper="0.0" lower="-1.047198" effort="1.0" velocity="6.5"/>
+  <dynamics damping="0.1"/>
 </joint>
 <joint name="Revolute_GRIPPER_R1" type="revolute">
@@ -534,4 +541,5 @@
   <axis xyz="-5e-06 -0.002097 0.999998"/>
   <limit upper="1.047198" lower="0.0" effort="1.0" velocity="6.5"/>
+  <dynamics damping="0.1"/>
 </joint>
 <joint name="rigid_GRIPPER_BASE_ARM_UPPER" type="fixed">
