Commit message: Fix JETANK drive system: replace JointController with DiffDrive, eliminate drift and veering
Root cause: Gazebo Harmonic's JointController (SetForce/PID) doesn't interact
with ground contact friction — wheels spin at target velocity but produce zero
traction (98% slip). Replaced with DiffDrive plugin which uses SetVelocityCommand
(motor constraint) that properly couples with the physics contact solver.

Key changes:
- Replace per-wheel JointController velocity plugins with DiffDrive plugin
- Align drive wheel axes (both +Y) so DiffDrive works correctly
- Symmetrize wheel joint positions to eliminate veering and idle drift
- Mirror left-side wheel visuals using right-side STL meshes (Y-flipped)
- Bridge /cmd_vel as Twist instead of per-wheel Float64 topics
- Remove cmd_vel_to_wheels node (DiffDrive handles kinematics)
- Zero gripper I-gain and increase arm joint damping to suppress drift
- Reduce free wheel damping (5.0 → 0.05) to eliminate rolling resistance
- Set sim-specific drive speed default (0.1 m/s vs 0.5 for real hardware)
- Fix angular velocity not to invert with wheels_inverted flag
- Disable self_collide on all links

File: JETANK_description/urdf/JETANK.xacro (robot description, xacro)
@@ -98,5 +98,5 @@
   </inertial>
   <visual>
-    <origin xyz="-0.05431 0.054968 0.052234" rpy="0 0 0"/>
+    <origin xyz="-0.05431 0.034968 0.052234" rpy="0 0 0"/>
     <geometry>
       <mesh filename="file://$(find JETANK_description)/meshes/FREE_WHEEL_L_1.stl" scale="0.001 0.001 0.001"/>
@@ -118,7 +118,7 @@
   </inertial>
   <visual>
-    <origin xyz="0.063868 -0.033862 0.052048" rpy="0 0 0"/>
-    <geometry>
-      <mesh filename="file://$(find JETANK_description)/meshes/FREE_WHEEL_R_1.stl" scale="0.001 0.001 0.001"/>
+    <origin xyz="-0.05431 -0.054968 0.052234" rpy="0 0 0"/>
+    <geometry>
+      <mesh filename="file://$(find JETANK_description)/meshes/FREE_WHEEL_L_1.stl" scale="0.001 -0.001 0.001"/>
     </geometry>
     <material name="wheel_material"/>
@@ -278,7 +278,7 @@
   </inertial>
   <visual>
-    <origin xyz="-0.054631 -0.033431 0.052049" rpy="0 0 0"/>
-    <geometry>
-      <mesh filename="file://$(find JETANK_description)/meshes/DRIVER_WHEEL_R_2.stl" scale="0.001 0.001 0.001"/>
+    <origin xyz="0.064189 -0.054537 0.052234" rpy="0 0 0"/>
+    <geometry>
+      <mesh filename="file://$(find JETANK_description)/meshes/DRIVER_WHEEL_L_1.stl" scale="0.001 -0.001 0.001"/>
     </geometry>
     <material name="wheel_material"/>
@@ -298,5 +298,5 @@
   </inertial>
   <visual>
-    <origin xyz="0.064189 0.054537 0.052234" rpy="0 0 0"/>
+    <origin xyz="0.064189 0.034537 0.052234" rpy="0 0 0"/>
     <geometry>
       <mesh filename="file://$(find JETANK_description)/meshes/DRIVER_WHEEL_L_1.stl" scale="0.001 0.001 0.001"/>
@@ -447,19 +447,19 @@
   <axis xyz="-4e-06 -0.002097 0.999998"/>
   <limit upper="1.8" lower="-1.8" effort="2.0" velocity="6.5"/>
-  <dynamics damping="0.5"/>
+  <dynamics damping="2.0"/>
 </joint>
 <joint name="revolute_FREE_WHEEL_LEFT" type="continuous">
-  <origin xyz="0.054304 -0.054100 -0.053366" rpy="0 0 0"/>
+  <origin xyz="0.054 -0.043 -0.053" rpy="0 0 0"/>
   <parent link="base_link"/>
   <child link="FREE_WHEEL_L_1"/>
   <axis xyz="0 1 0"/>
-  <dynamics damping="0.01"/>
+  <dynamics damping="0.05" friction="0.02"/>
 </joint>
 <joint name="revolute_FREE_WHEEL_RIGHT" type="continuous">
-  <origin xyz="-0.063847 0.033000 -0.053410" rpy="0 0 0"/>
+  <origin xyz="0.054 0.043 -0.053" rpy="0 0 0"/>
   <parent link="base_link"/>
   <child link="FREE_WHEEL_R_1"/>
   <axis xyz="0 -1 0"/>
-  <dynamics damping="0.01"/>
+  <dynamics damping="0.05" friction="0.02"/>
 </joint>
 <joint name="rigid_CAMERA_CAMERA_HOLDER" type="fixed">
@@ -474,5 +474,5 @@
   <axis xyz="0 1 0"/>
   <limit upper="1.0" lower="-1.0" effort="2.0" velocity="6.5"/>
-  <dynamics damping="0.2"/>
+  <dynamics damping="1.0"/>
 </joint>
 <joint name="revolute_GRIPPER_L1" type="revolute">
@@ -498,5 +498,5 @@
   <axis xyz="-0.003633 -0.999991 -0.002097"/>
   <limit upper="1.0" lower="-1.548620" effort="2.0" velocity="6.5"/>
-  <dynamics damping="0.3"/>
+  <dynamics damping="2.0"/>
 </joint>
 <joint name="Revolute_SERVO_LOWER" type="revolute">
@@ -506,5 +506,5 @@
   <axis xyz="-0.003633 -0.999991 -0.002097"/>
   <limit upper="1.574492" lower="-1.892348" effort="2.0" velocity="6.5"/>
-  <dynamics damping="0.3"/>
+  <dynamics damping="2.0"/>
 </joint>
 <joint name="Rigid_SERVO_LOWER_ARM_LOWER" type="fixed">
@@ -514,16 +514,18 @@
 </joint>
 <joint name="Revolute_DRIVING_WHEEL_R" type="continuous">
-  <origin xyz="0.054634 0.032570 -0.050948" rpy="0 0 0"/>
+  <origin xyz="-0.060 0.043 -0.051" rpy="0 0 0"/>
   <parent link="base_link"/>
   <child link="DRIVER_WHEEL_R_2"/>
-  <axis xyz="0 -1 0"/>
+  <axis xyz="0 1 0"/>
   <limit effort="100" velocity="100"/>
+  <dynamics damping="50.0" friction="5.0"/>
 </joint>
 <joint name="Revolute_DRIVING_WHEEL_L" type="continuous">
-  <origin xyz="-0.064218 -0.053670 -0.050868" rpy="0 0 0"/>
+  <origin xyz="-0.060 -0.043 -0.051" rpy="0 0 0"/>
   <parent link="base_link"/>
   <child link="DRIVER_WHEEL_L_1"/>
   <axis xyz="0 1 0"/>
   <limit effort="100" velocity="100"/>
+  <dynamics damping="50.0" friction="5.0"/>
 </joint>
 <joint name="Revolute_GRIPPER_R2" type="revolute">
