Commit message: Update camera holder joint from fixed to revolute

File: JETANK_description/urdf/JETANK.urdf (robot description, URDF)
Before this commit: robot JETANK, 21 links, 20 joints
Links:
- link ANTENNA_L_1: geometry collision mesh filename=file:///home/ubuntu/ros2_ws/install/JETANK_description/shar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 scale=0.001 0.001 0.001; visual mesh filename=file:///home/ubuntu/ros2_ws/install/JETANK_description/shar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 scale=0.001 0.001 0.001
- link ANTENNA_R_2: geometry collision mesh filename=file:///home/ubuntu/ros2_ws/install/JETANK_description/shar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 scale=0.001 0.001 0.001; visual mesh filename=file:///home/ubuntu/ros2_ws/install/JETANK_description/shar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 scale=0.001 0.001 0.001
- link ARM_LOWER_1: geometry collision mesh filename=file:///home/ubuntu/ros2_ws/install/JETANK_description/shar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 scale=0.001 0.001 0.001; visual mesh filename=file:///home/ubuntu/ros2_ws/install/JETANK_description/shar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 scale=0.001 0.001 0.001
- link ARM_MIDDLE_2: geometry collision mesh filename=file:///home/ubuntu/ros2_ws/install/JETANK_description/shar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 scale=0.001 0.001 0.001; visual mesh filename=file:///home/ubuntu/ros2_ws/install/JETANK_description/shar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 scale=0.001 0.001 0.001
- link ARM_UPPER_1: geometry collision mesh filename=file:///home/ubuntu/ros2_ws/install/JETANK_description/shar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 scale=0.001 0.001 0.001; visual mesh filename=file:///home/ubuntu/ros2_ws/install/JETANK_description/shar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 scale=0.001 0.001 0.001
- link BEARING_1: geometry collision mesh filename=file:///home/ubuntu/ros2_ws/install/JETANK_description/shar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 scale=0.001 0.001 0.001; visual mesh filename=file:///home/ubuntu/ros2_ws/install/JETANK_description/shar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 scale=0.001 0.001 0.001
- link CAMERA_1: geometry collision mesh filename=file:///home/ubuntu/ros2_ws/install/JETANK_description/shar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 scale=0.001 0.001 0.001; visual mesh filename=file:///home/ubuntu/ros2_ws/install/JETANK_description/shar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 scale=0.001 0.001 0.001
- link CAM_HOLDER_1: geometry collision mesh filename=file:///home/ubuntu/ros2_ws/install/JETANK_description/shar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 scale=0.001 0.001 0.001; visual mesh filename=file:///home/ubuntu/ros2_ws/install/JETANK_description/shar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 scale=0.001 0.001 0.001
- link DRIVER_WHEEL_L_1: geometry collision mesh filename=file:///home/ubuntu/ros2_ws/install/JETANK_description/shar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 scale=0.001 0.001 0.001; visual mesh filename=file:///home/ubuntu/ros2_ws/install/JETANK_description/shar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 scale=0.001 0.001 0.001
- link DRIVER_WHEEL_R_2: geometry collision mesh filename=file:///home/ubuntu/ros2_ws/install/JETANK_description/shar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 scale=0.001 0.001 0.001; visual mesh filename=file:///home/ubuntu/ros2_ws/install/JETANK_description/shar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 scale=0.001 0.001 0.001
- link FREE_WHEEL_L_1: geometry collision mesh filename=file:///home/ubuntu/ros2_ws/install/JETANK_description/shar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 scale=0.001 0.001 0.001; visual mesh filename=file:///home/ubuntu/ros2_ws/install/JETANK_description/shar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 scale=0.001 0.001 0.001
- link FREE_WHEEL_R_1: geometry collision mesh filename=file:///home/ubuntu/ros2_ws/install/JETANK_description/shar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 scale=0.001 0.001 0.001; visual mesh filename=file:///home/ubuntu/ros2_ws/install/JETANK_description/shar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 scale=0.001 0.001 0.001
- link GRIPPER_BASE_1: geometry collision mesh filename=file:///home/ubuntu/ros2_ws/install/JETANK_description/shar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 scale=0.001 0.001 0.001; visual mesh filename=file:///home/ubuntu/ros2_ws/install/JETANK_description/shar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 scale=0.001 0.001 0.001
- link GRIPPER_L1_1: geometry collision mesh filename=file:///home/ubuntu/ros2_ws/install/JETANK_description/shar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 scale=0.001 0.001 0.001; visual mesh filename=file:///home/ubuntu/ros2_ws/install/JETANK_description/shar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 scale=0.001 0.001 0.001
- link GRIPPER_L2_1: geometry collision mesh filename=file:///home/ubuntu/ros2_ws/install/JETANK_description/shar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 scale=0.001 0.001 0.001; visual mesh filename=file:///home/ubuntu/ros2_ws/install/JETANK_description/shar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 scale=0.001 0.001 0.001
- link GRIPPER_R1_1: geometry collision mesh filename=file:///home/ubuntu/ros2_ws/install/JETANK_description/shar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 scale=0.001 0.001 0.001; visual mesh filename=file:///home/ubuntu/ros2_ws/install/JETANK_description/shar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 scale=0.001 0.001 0.001
- link GRIPPER_R2_1: geometry collision mesh filename=file:///home/ubuntu/ros2_ws/install/JETANK_description/shar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 scale=0.001 0.001 0.001; visual mesh filename=file:///home/ubuntu/ros2_ws/install/JETANK_description/shar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 scale=0.001 0.001 0.001
- link SERVO_LOWER_1: geometry collision mesh filename=file:///home/ubuntu/ros2_ws/install/JETANK_description/shar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 scale=0.001 0.001 0.001; visual mesh filename=file:///home/ubuntu/ros2_ws/install/JETANK_description/shar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 scale=0.001 0.001 0.001
- link SERVO_UPPER_1: geometry collision mesh filename=file:///home/ubuntu/ros2_ws/install/JETANK_description/shar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 scale=0.001 0.001 0.001; visual mesh filename=file:///home/ubuntu/ros2_ws/install/JETANK_description/shar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 scale=0.001 0.001 0.001
- link base_link: geometry collision mesh filename=file:///home/ubuntu/ros2_ws/install/JETANK_description/shar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 scale=0.001 0.001 0.001; visual mesh filename=file:///home/ubuntu/ros2_ws/install/JETANK_description/shar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 scale=0.001 0.001 0.001

File: JETANK_description/urdf/JETANK.xacro (robot description, xacro)
@@ -15,5 +15,5 @@
       <mesh filename="file://$(find JETANK_description)/meshes/base_link.stl" scale="0.001 0.001 0.001"/>
     </geometry>
-    <material name="base_link_material"/>
+    <material name="silver"/>
   </visual>
   <collision>
@@ -35,5 +35,5 @@
       <mesh filename="file://$(find JETANK_description)/meshes/ANTENNA_L_1.stl" scale="0.001 0.001 0.001"/>
     </geometry>
-    <material name="antenna_material"/>
+    <material name="silver"/>
   </visual>
   <collision>
@@ -55,5 +55,5 @@
       <mesh filename="file://$(find JETANK_description)/meshes/BEARING_1.stl" scale="0.001 0.001 0.001"/>
     </geometry>
-    <material name="bearing_material"/>
+    <material name="silver"/>
   </visual>
   <collision>
@@ -75,5 +75,5 @@
       <mesh filename="file://$(find JETANK_description)/meshes/ARM_LOWER_1.stl" scale="0.001 0.001 0.001"/>
     </geometry>
-    <material name="arm_material"/>
+    <material name="silver"/>
   </visual>
   <collision>
@@ -95,5 +95,5 @@
       <mesh filename="file://$(find JETANK_description)/meshes/FREE_WHEEL_L_1.stl" scale="0.001 0.001 0.001"/>
     </geometry>
-    <material name="wheel_material"/>
+    <material name="silver"/>
   </visual>
   <collision>
@@ -115,5 +115,5 @@
       <mesh filename="file://$(find JETANK_description)/meshes/FREE_WHEEL_R_1.stl" scale="0.001 0.001 0.001"/>
     </geometry>
-    <material name="wheel_material"/>
+    <material name="silver"/>
   </visual>
   <collision>
@@ -135,5 +135,5 @@
       <mesh filename="file://$(find JETANK_description)/meshes/CAMERA_1.stl" scale="0.001 0.001 0.001"/>
     </geometry>
-    <material name="camera_material"/>
+    <material name="silver"/>
   </visual>
   <collision>
@@ -155,5 +155,5 @@
       <mesh filename="file://$(find JETANK_description)/meshes/CAM_HOLDER_1.stl" scale="0.001 0.001 0.001"/>
     </geometry>
-    <material name="camera_holder_material"/>
+    <material name="silver"/>
   </visual>
   <collision>
@@ -175,5 +175,5 @@
       <mesh filename="file://$(find JETANK_description)/meshes/GRIPPER_L1_1.stl" scale="0.001 0.001 0.001"/>
     </geometry>
-    <material name="gripper_material"/>
+    <material name="silver"/>
   </visual>
   <collision>
@@ -195,5 +195,5 @@
       <mesh filename="file://$(find JETANK_description)/meshes/GRIPPER_L2_1.stl" scale="0.001 0.001 0.001"/>
     </geometry>
-    <material name="gripper_material"/>
+    <material name="silver"/>
   </visual>
   <collision>
@@ -215,5 +215,5 @@
       <mesh filename="file://$(find JETANK_description)/meshes/SERVO_UPPER_1.stl" scale="0.001 0.001 0.001"/>
     </geometry>
-    <material name="servo_material"/>
+    <material name="silver"/>
   </visual>
   <collision>
@@ -235,5 +235,5 @@
       <mesh filename="file://$(find JETANK_description)/meshes/ARM_MIDDLE_2.stl" scale="0.001 0.001 0.001"/>
     </geometry>
-    <material name="arm_material"/>
+    <material name="silver"/>
   </visual>
   <collision>
@@ -255,5 +255,5 @@
       <mesh filename="file://$(find JETANK_description)/meshes/SERVO_LOWER_1.stl" scale="0.001 0.001 0.001"/>
     </geometry>
-    <material name="servo_material"/>
+    <material name="silver"/>
   </visual>
   <collision>
@@ -275,5 +275,5 @@
       <mesh filename="file://$(find JETANK_description)/meshes/DRIVER_WHEEL_R_2.stl" scale="0.001 0.001 0.001"/>
     </geometry>
-    <material name="wheel_material"/>
+    <material name="silver"/>
   </visual>
   <collision>
@@ -295,5 +295,5 @@
       <mesh filename="file://$(find JETANK_description)/meshes/DRIVER_WHEEL_L_1.stl" scale="0.001 0.001 0.001"/>
     </geometry>
-    <material name="wheel_material"/>
+    <material name="silver"/>
   </visual>
   <collision>
@@ -315,5 +315,5 @@
       <mesh filename="file://$(find JETANK_description)/meshes/GRIPPER_R2_1.stl" scale="0.001 0.001 0.001"/>
     </geometry>
-    <material name="gripper_material"/>
+    <material name="silver"/>
   </visual>
   <collision>
@@ -335,5 +335,5 @@
       <mesh filename="file://$(find JETANK_description)/meshes/GRIPPER_R1_1.stl" scale="0.001 0.001 0.001"/>
     </geometry>
-    <material name="gripper_material"/>
+    <material name="silver"/>
   </visual>
   <collision>
@@ -355,5 +355,5 @@
       <mesh filename="file://$(find JETANK_description)/meshes/GRIPPER_BASE_1.stl" scale="0.001 0.001 0.001"/>
     </geometry>
-    <material name="gripper_material"/>
+    <material name="silver"/>
   </visual>
   <collision>
@@ -375,5 +375,5 @@
       <box size="0.01 0.01 0.01"/>
     </geometry>
-    <material name="gripper_material"/>
+    <material name="silver"/>
   </visual>
   <collision>
@@ -395,5 +395,5 @@
       <mesh filename="file://$(find JETANK_description)/meshes/ARM_UPPER_1.stl" scale="0.001 0.001 0.001"/>
     </geometry>
-    <material name="arm_material"/>
+    <material name="silver"/>
   </visual>
   <collision>
@@ -415,5 +415,5 @@
       <mesh filename="file://$(find JETANK_description)/meshes/ANTENNA_R_2.stl" scale="0.001 0.001 0.001"/>
     </geometry>
-    <material name="antenna_material"/>
+    <material name="silver"/>
   </visual>
   <collision>
@@ -460,8 +460,10 @@
   <child link="CAMERA_1"/>
 </joint>
-<joint name="rigid_CAMERA_HOLDER_ARM_LOWER" type="fixed">
+<joint name="revolute_CAMERA_HOLDER_ARM_LOWER" type="revolute">
   <origin xyz="-0.0248 1.8e-05 0.034381" rpy="0 0 0"/>
   <parent link="ARM_LOWER_1"/>
   <child link="CAM_HOLDER_1"/>
+  <axis xyz="0 1 0"/>
+  <limit upper="0.785398" lower="-0.785398" effort="100" velocity="100"/>
 </joint>
 <joint name="revolute_GRIPPER_L1" type="revolute">

Commit message: Update format for isaacsim import

File: JETANK_description/urdf/JETANK.urdf (robot description, URDF)
Before this commit: robot JETANK, 21 links, 20 joints
Links:
- link ANTENNA_L_1: geometry collision mesh filename=file:///home/aaugus11/ros2_ws/install/JETANK_description/sh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 scale=0.001 0.001 0.001; visual mesh filename=file:///home/aaugus11/ros2_ws/install/JETANK_description/sh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 scale=0.001 0.001 0.001
- link ANTENNA_R_2: geometry collision mesh filename=file:///home/aaugus11/ros2_ws/install/JETANK_description/sh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 scale=0.001 0.001 0.001; visual mesh filename=file:///home/aaugus11/ros2_ws/install/JETANK_description/sh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 scale=0.001 0.001 0.001
- link ARM_LOWER_1: geometry collision mesh filename=file:///home/aaugus11/ros2_ws/install/JETANK_description/sh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 scale=0.001 0.001 0.001; visual mesh filename=file:///home/aaugus11/ros2_ws/install/JETANK_description/sh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 scale=0.001 0.001 0.001
- link ARM_MIDDLE_2: geometry collision mesh filename=file:///home/aaugus11/ros2_ws/install/JETANK_description/sh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 scale=0.001 0.001 0.001; visual mesh filename=file:///home/aaugus11/ros2_ws/install/JETANK_description/sh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 scale=0.001 0.001 0.001
- link ARM_UPPER_1: geometry collision mesh filename=file:///home/aaugus11/ros2_ws/install/JETANK_description/sh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 scale=0.001 0.001 0.001; visual mesh filename=file:///home/aaugus11/ros2_ws/install/JETANK_description/sh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 scale=0.001 0.001 0.001
- link BEARING_1: geometry collision mesh filename=file:///home/aaugus11/ros2_ws/install/JETANK_description/sh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 scale=0.001 0.001 0.001; visual mesh filename=file:///home/aaugus11/ros2_ws/install/JETANK_description/sh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 scale=0.001 0.001 0.001
- link CAMERA_1: geometry collision mesh filename=file:///home/aaugus11/ros2_ws/install/JETANK_description/sh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 scale=0.001 0.001 0.001; visual mesh filename=file:///home/aaugus11/ros2_ws/install/JETANK_description/sh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 scale=0.001 0.001 0.001
- link CAM_HOLDER_1: geometry collision mesh filename=file:///home/aaugus11/ros2_ws/install/JETANK_description/sh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 scale=0.001 0.001 0.001; visual mesh filename=file:///home/aaugus11/ros2_ws/install/JETANK_description/sh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 scale=0.001 0.001 0.001
- link DRIVER_WHEEL_L_1: geometry collision mesh filename=file:///home/aaugus11/ros2_ws/install/JETANK_description/sh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 scale=0.001 0.001 0.001; visual mesh filename=file:///home/aaugus11/ros2_ws/install/JETANK_description/sh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 scale=0.001 0.001 0.001
- link DRIVER_WHEEL_R_2: geometry collision mesh filename=file:///home/aaugus11/ros2_ws/install/JETANK_description/sh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 scale=0.001 0.001 0.001; visual mesh filename=file:///home/aaugus11/ros2_ws/install/JETANK_description/sh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 scale=0.001 0.001 0.001
- link FREE_WHEEL_L_1: geometry collision mesh filename=file:///home/aaugus11/ros2_ws/install/JETANK_description/sh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 scale=0.001 0.001 0.001; visual mesh filename=file:///home/aaugus11/ros2_ws/install/JETANK_description/sh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 scale=0.001 0.001 0.001
- link FREE_WHEEL_R_1: geometry collision mesh filename=file:///home/aaugus11/ros2_ws/install/JETANK_description/sh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 scale=0.001 0.001 0.001; visual mesh filename=file:///home/aaugus11/ros2_ws/install/JETANK_description/sh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 scale=0.001 0.001 0.001
- link GRIPPER_BASE_1: geometry collision mesh filename=file:///home/aaugus11/ros2_ws/install/JETANK_description/sh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 scale=0.001 0.001 0.001; visual mesh filename=file:///home/aaugus11/ros2_ws/install/JETANK_description/sh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 scale=0.001 0.001 0.001
- link GRIPPER_L1_1: geometry collision mesh filename=file:///home/aaugus11/ros2_ws/install/JETANK_description/sh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 scale=0.001 0.001 0.001; visual mesh filename=file:///home/aaugus11/ros2_ws/install/JETANK_description/sh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 scale=0.001 0.001 0.001
- link GRIPPER_L2_1: geometry collision mesh filename=file:///home/aaugus11/ros2_ws/install/JETANK_description/sh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 scale=0.001 0.001 0.001; visual mesh filename=file:///home/aaugus11/ros2_ws/install/JETANK_description/sh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 scale=0.001 0.001 0.001
- link GRIPPER_R1_1: geometry collision mesh filename=file:///home/aaugus11/ros2_ws/install/JETANK_description/sh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 scale=0.001 0.001 0.001; visual mesh filename=file:///home/aaugus11/ros2_ws/install/JETANK_description/sh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 scale=0.001 0.001 0.001
- link GRIPPER_R2_1: geometry collision mesh filename=file:///home/aaugus11/ros2_ws/install/JETANK_description/sh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 scale=0.001 0.001 0.001; visual mesh filename=file:///home/aaugus11/ros2_ws/install/JETANK_description/sh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 scale=0.001 0.001 0.001
- link SERVO_LOWER_1: geometry collision mesh filename=file:///home/aaugus11/ros2_ws/install/JETANK_description/sh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 scale=0.001 0.001 0.001; visual mesh filename=file:///home/aaugus11/ros2_ws/install/JETANK_description/sh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 scale=0.001 0.001 0.001
- link SERVO_UPPER_1: geometry collision mesh filename=file:///home/aaugus11/ros2_ws/install/JETANK_description/sh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 scale=0.001 0.001 0.001; visual mesh filename=file:///home/aaugus11/ros2_ws/install/JETANK_description/sh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 scale=0.001 0.001 0.001
- link base_link: geometry collision mesh filename=file:///home/aaugus11/ros2_ws/install/JETANK_description/sh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 scale=0.001 0.001 0.001; visual mesh filename=file:///home/aaugus11/ros2_ws/install/JETANK_description/sh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 scale=0.001 0.001 0.001
Joints:
- removed joint rigid_CAMERA_HOLDER_ARM_LOWER
- added joint revolute_CAMERA_HOLDER_ARM_LOWER: type revolute, parent ARM_LOWER_1, child CAM_HOLDER_1, origin xyz=-0.0248 1.8e-05 0.034381 rpy=0 0 0, axis 0 1 0, limit lower=-0.785398 upper=0.785398 effort=100 velocity=100

File: JETANK_description/urdf/JETANK.xacro (robot description, xacro)
@@ -15,5 +15,5 @@
       <mesh filename="file://$(find JETANK_description)/meshes/base_link.stl" scale="0.001 0.001 0.001"/>
     </geometry>
-    <material name="silver"/>
+    <material name="base_link_material"/>
   </visual>
   <collision>
@@ -35,5 +35,5 @@
       <mesh filename="file://$(find JETANK_description)/meshes/ANTENNA_L_1.stl" scale="0.001 0.001 0.001"/>
     </geometry>
-    <material name="silver"/>
+    <material name="antenna_material"/>
   </visual>
   <collision>
@@ -55,5 +55,5 @@
       <mesh filename="file://$(find JETANK_description)/meshes/BEARING_1.stl" scale="0.001 0.001 0.001"/>
     </geometry>
-    <material name="silver"/>
+    <material name="bearing_material"/>
   </visual>
   <collision>
@@ -75,5 +75,5 @@
       <mesh filename="file://$(find JETANK_description)/meshes/ARM_LOWER_1.stl" scale="0.001 0.001 0.001"/>
     </geometry>
-    <material name="silver"/>
+    <material name="arm_material"/>
   </visual>
   <collision>
@@ -95,5 +95,5 @@
       <mesh filename="file://$(find JETANK_description)/meshes/FREE_WHEEL_L_1.stl" scale="0.001 0.001 0.001"/>
     </geometry>
-    <material name="silver"/>
+    <material name="wheel_material"/>
   </visual>
   <collision>
@@ -115,5 +115,5 @@
       <mesh filename="file://$(find JETANK_description)/meshes/FREE_WHEEL_R_1.stl" scale="0.001 0.001 0.001"/>
     </geometry>
-    <material name="silver"/>
+    <material name="wheel_material"/>
   </visual>
   <collision>
@@ -135,5 +135,5 @@
       <mesh filename="file://$(find JETANK_description)/meshes/CAMERA_1.stl" scale="0.001 0.001 0.001"/>
     </geometry>
-    <material name="silver"/>
+    <material name="camera_material"/>
   </visual>
   <collision>
@@ -155,5 +155,5 @@
       <mesh filename="file://$(find JETANK_description)/meshes/CAM_HOLDER_1.stl" scale="0.001 0.001 0.001"/>
     </geometry>
-    <material name="silver"/>
+    <material name="camera_holder_material"/>
   </visual>
   <collision>
@@ -175,5 +175,5 @@
       <mesh filename="file://$(find JETANK_description)/meshes/GRIPPER_L1_1.stl" scale="0.001 0.001 0.001"/>
     </geometry>
-    <material name="silver"/>
+    <material name="gripper_material"/>
   </visual>
   <collision>
@@ -195,5 +195,5 @@
       <mesh filename="file://$(find JETANK_description)/meshes/GRIPPER_L2_1.stl" scale="0.001 0.001 0.001"/>
     </geometry>
-    <material name="silver"/>
+    <material name="gripper_material"/>
   </visual>
   <collision>
@@ -215,5 +215,5 @@
       <mesh filename="file://$(find JETANK_description)/meshes/SERVO_UPPER_1.stl" scale="0.001 0.001 0.001"/>
     </geometry>
-    <material name="silver"/>
+    <material name="servo_material"/>
   </visual>
   <collision>
@@ -235,5 +235,5 @@
       <mesh filename="file://$(find JETANK_description)/meshes/ARM_MIDDLE_2.stl" scale="0.001 0.001 0.001"/>
     </geometry>
-    <material name="silver"/>
+    <material name="arm_material"/>
   </visual>
   <collision>
@@ -255,5 +255,5 @@
       <mesh filename="file://$(find JETANK_description)/meshes/SERVO_LOWER_1.stl" scale="0.001 0.001 0.001"/>
     </geometry>
-    <material name="silver"/>
+    <material name="servo_material"/>
   </visual>
   <collision>
@@ -275,5 +275,5 @@
       <mesh filename="file://$(find JETANK_description)/meshes/DRIVER_WHEEL_R_2.stl" scale="0.001 0.001 0.001"/>
     </geometry>
-    <material name="silver"/>
+    <material name="wheel_material"/>
   </visual>
   <collision>
@@ -295,5 +295,5 @@
       <mesh filename="file://$(find JETANK_description)/meshes/DRIVER_WHEEL_L_1.stl" scale="0.001 0.001 0.001"/>
     </geometry>
-    <material name="silver"/>
+    <material name="wheel_material"/>
   </visual>
   <collision>
@@ -315,5 +315,5 @@
       <mesh filename="file://$(find JETANK_description)/meshes/GRIPPER_R2_1.stl" scale="0.001 0.001 0.001"/>
     </geometry>
-    <material name="silver"/>
+    <material name="gripper_material"/>
   </visual>
   <collision>
@@ -335,5 +335,5 @@
       <mesh filename="file://$(find JETANK_description)/meshes/GRIPPER_R1_1.stl" scale="0.001 0.001 0.001"/>
     </geometry>
-    <material name="silver"/>
+    <material name="gripper_material"/>
   </visual>
   <collision>
@@ -355,5 +355,5 @@
       <mesh filename="file://$(find JETANK_description)/meshes/GRIPPER_BASE_1.stl" scale="0.001 0.001 0.001"/>
     </geometry>
-    <material name="silver"/>
+    <material name="gripper_material"/>
   </visual>
   <collision>
@@ -375,5 +375,5 @@
       <box size="0.01 0.01 0.01"/>
     </geometry>
-    <material name="silver"/>
+    <material name="gripper_material"/>
   </visual>
   <collision>
@@ -395,5 +395,5 @@
       <mesh filename="file://$(find JETANK_description)/meshes/ARM_UPPER_1.stl" scale="0.001 0.001 0.001"/>
     </geometry>
-    <material name="silver"/>
+    <material name="arm_material"/>
   </visual>
   <collision>
@@ -415,5 +415,5 @@
       <mesh filename="file://$(find JETANK_description)/meshes/ANTENNA_R_2.stl" scale="0.001 0.001 0.001"/>
     </geometry>
-    <material name="silver"/>
+    <material name="antenna_material"/>
   </visual>
   <collision>
