Commit message: Update joint limits to match real world

File: JETANK_description/urdf/JETANK.urdf (robot description, URDF)
Before this commit: robot JETANK, 21 links, 20 joints
Joints:
- joint Revolute_SERVO_LOWER: limit lower=0.0 upper=1.570796 effort=100 velocity=100 -> lower=-1.892348 upper=1.574492 effort=100 velocity=100
- joint Revolute_SERVO_UPPER: limit lower=-3.1418 upper=0.785594 effort=100 velocity=100 -> lower=-1.548620 upper=1.0 effort=100 velocity=100
- joint revolute_BEARING: limit lower=-1.5708 upper=1.5708 effort=100 velocity=100 -> lower=-1.8 upper=1.8 effort=100 velocity=100
- joint revolute_CAMERA_HOLDER_ARM_LOWER: limit lower=-0.785398 upper=0.785398 effort=100 velocity=100 -> lower=-1.0 upper=1.0 effort=100 velocity=100

File: JETANK_description/urdf/JETANK.xacro (robot description, xacro)
@@ -439,5 +439,5 @@
   <child link="ARM_LOWER_1"/>
   <axis xyz="-4e-06 -0.002097 0.999998"/>
-  <limit upper="1.5708" lower="-1.5708" effort="100" velocity="100"/>
+  <limit upper="1.8" lower="-1.8" effort="100" velocity="100"/>
 </joint>
 <joint name="revolute_FREE_WHEEL_LEFT" type="revolute">
@@ -465,5 +465,5 @@
   <child link="CAM_HOLDER_1"/>
   <axis xyz="0 1 0"/>
-  <limit upper="0.785398" lower="-0.785398" effort="100" velocity="100"/>
+  <limit upper="1.0" lower="-1.0" effort="100" velocity="100"/>
 </joint>
 <joint name="revolute_GRIPPER_L1" type="revolute">
@@ -486,5 +486,5 @@
   <child link="SERVO_UPPER_1"/>
   <axis xyz="-0.003633 -0.999991 -0.002097"/>
-  <limit upper="0.785594" lower="-3.1418" effort="100" velocity="100"/>
+  <limit upper="1.0" lower="-1.548620" effort="100" velocity="100"/>
 </joint>
 <joint name="Revolute_SERVO_LOWER" type="revolute">
@@ -493,5 +493,5 @@
   <child link="ARM_MIDDLE_2"/>
   <axis xyz="-0.003633 -0.999991 -0.002097"/>
-  <limit upper="1.570796" lower="0.0" effort="100" velocity="100"/>
+  <limit upper="1.574492" lower="-1.892348" effort="100" velocity="100"/>
 </joint>
 <joint name="Rigid_SERVO_LOWER_ARM_LOWER" type="fixed">

Commit message: update gripper range to match real world

File: JETANK_description/urdf/JETANK.urdf (robot description, URDF)
Before this commit: robot JETANK, 21 links, 20 joints
Joints:
- joint Revolute_GRIPPER_R1: limit lower=0.0 upper=0.785398 effort=100 velocity=100 -> lower=0.0 upper=1.047198 effort=100 velocity=100
- joint Revolute_GRIPPER_R2: limit lower=-0.785398 upper=0.0 effort=100 velocity=100 -> lower=-1.047198 upper=0.0 effort=100 velocity=100
- joint revolute_GRIPPER_L1: limit lower=-0.785398 upper=0.0 effort=100 velocity=100 -> lower=-1.047198 upper=0.0 effort=100 velocity=100
- joint revolute_GRIPPER_L2: limit lower=-0.785398 upper=0.0 effort=100 velocity=100 -> lower=-1.047198 upper=0.0 effort=100 velocity=100

File: JETANK_description/urdf/JETANK.xacro (robot description, xacro)
@@ -472,5 +472,5 @@
   <child link="GRIPPER_L1_1"/>
   <axis xyz="-5e-06 -0.002097 0.999998"/>
-  <limit upper="0.0" lower="-0.785398" effort="100" velocity="100"/>
+  <limit upper="0.0" lower="-1.047198" effort="100" velocity="100"/>
 </joint>
 <joint name="revolute_GRIPPER_L2" type="revolute">
@@ -479,5 +479,5 @@
   <child link="GRIPPER_L2_1"/>
   <axis xyz="5e-06 0.002097 -0.999998"/>
-  <limit upper="0.0" lower="-0.785398" effort="100" velocity="100"/>
+  <limit upper="0.0" lower="-1.047198" effort="100" velocity="100"/>
 </joint>
 <joint name="Revolute_SERVO_UPPER" type="revolute">
@@ -519,5 +519,5 @@
   <child link="GRIPPER_R2_1"/>
   <axis xyz="-5e-06 -0.002097 0.999998"/>
-  <limit upper="0.0" lower="-0.785398" effort="100" velocity="100"/>
+  <limit upper="0.0" lower="-1.047198" effort="100" velocity="100"/>
 </joint>
 <joint name="Revolute_GRIPPER_R1" type="revolute">
@@ -526,5 +526,5 @@
   <child link="GRIPPER_R1_1"/>
   <axis xyz="-5e-06 -0.002097 0.999998"/>
-  <limit upper="0.785398" lower="0.0" effort="100" velocity="100"/>
+  <limit upper="1.047198" lower="0.0" effort="100" velocity="100"/>
 </joint>
 <joint name="rigid_GRIPPER_BASE_ARM_UPPER" type="fixed">

Commit message: Fix depth camera, add headless Gazebo, make legos static
- Add CAMERA_SENSOR_FRAME link 20mm forward to clear depth camera housing
- Offset both RGB and depth sensors to CAMERA_SENSOR_FRAME
- camera_pose_publisher uses CAMERA_SENSOR_FRAME
- Reduce depth far clip to 2m, disable anti-aliasing for clean depth
- Add headless launch arg (headless:=true runs server-only)
- Remove hardcoded DISPLAY env var from launch file
- Make lego bricks static at resting positions (no physics settling)
- Convert URDF mesh paths from absolute to package:// URIs

File: JETANK_description/urdf/JETANK.urdf (robot description, URDF)
Before this commit: robot JETANK, 21 links, 20 joints
Links:
- link ANTENNA_L_1: geometry collision mesh filename=package://JETANK_description/meshes/ANTENNA_L_1.stl scale=0.001 0.001 0.001; visual mesh filename=package://JETANK_description/meshes/ANTENNA_L_1.stl scale=0.001 0.001 0.001
- link ANTENNA_R_2: geometry collision mesh filename=package://JETANK_description/meshes/ANTENNA_R_2.stl scale=0.001 0.001 0.001; visual mesh filename=package://JETANK_description/meshes/ANTENNA_R_2.stl scale=0.001 0.001 0.001
- link ARM_LOWER_1: geometry collision mesh filename=package://JETANK_description/meshes/ARM_LOWER_1.stl scale=0.001 0.001 0.001; visual mesh filename=package://JETANK_description/meshes/ARM_LOWER_1.stl scale=0.001 0.001 0.001
- link ARM_MIDDLE_2: geometry collision mesh filename=package://JETANK_description/meshes/ARM_MIDDLE_2.stl scale=0.001 0.001 0.001; visual mesh filename=package://JETANK_description/meshes/ARM_MIDDLE_2.stl scale=0.001 0.001 0.001
- link ARM_UPPER_1: geometry collision mesh filename=package://JETANK_description/meshes/ARM_UPPER_1.stl scale=0.001 0.001 0.001; visual mesh filename=package://JETANK_description/meshes/ARM_UPPER_1.stl scale=0.001 0.001 0.001
- link BEARING_1: geometry collision mesh filename=package://JETANK_description/meshes/BEARING_1.stl scale=0.001 0.001 0.001; visual mesh filename=package://JETANK_description/meshes/BEARING_1.stl scale=0.001 0.001 0.001
- link CAMERA_1: geometry collision mesh filename=package://JETANK_description/meshes/CAMERA_1.stl scale=0.001 0.001 0.001; visual mesh filename=package://JETANK_description/meshes/CAMERA_1.stl scale=0.001 0.001 0.001
- link CAM_HOLDER_1: geometry collision mesh filename=package://JETANK_description/meshes/CAM_HOLDER_1.stl scale=0.001 0.001 0.001; visual mesh filename=package://JETANK_description/meshes/CAM_HOLDER_1.stl scale=0.001 0.001 0.001
- link DRIVER_WHEEL_L_1: geometry collision mesh filename=package://JETANK_description/meshes/DRIVER_WHEEL_L_1.stl scale=0.001 0.001 0.001; visual mesh filename=package://JETANK_description/meshes/DRIVER_WHEEL_L_1.stl scale=0.001 0.001 0.001
- link DRIVER_WHEEL_R_2: geometry collision mesh filename=package://JETANK_description/meshes/DRIVER_WHEEL_R_2.stl scale=0.001 0.001 0.001; visual mesh filename=package://JETANK_description/meshes/DRIVER_WHEEL_R_2.stl scale=0.001 0.001 0.001
- link FREE_WHEEL_L_1: geometry collision mesh filename=package://JETANK_description/meshes/FREE_WHEEL_L_1.stl scale=0.001 0.001 0.001; visual mesh filename=package://JETANK_description/meshes/FREE_WHEEL_L_1.stl scale=0.001 0.001 0.001
- link FREE_WHEEL_R_1: geometry collision mesh filename=package://JETANK_description/meshes/FREE_WHEEL_R_1.stl scale=0.001 0.001 0.001; visual mesh filename=package://JETANK_description/meshes/FREE_WHEEL_R_1.stl scale=0.001 0.001 0.001
- link GRIPPER_BASE_1: geometry collision mesh filename=package://JETANK_description/meshes/GRIPPER_BASE_1.stl scale=0.001 0.001 0.001; visual mesh filename=package://JETANK_description/meshes/GRIPPER_BASE_1.stl scale=0.001 0.001 0.001
- link GRIPPER_L1_1: geometry collision mesh filename=package://JETANK_description/meshes/GRIPPER_L1_1.stl scale=0.001 0.001 0.001; visual mesh filename=package://JETANK_description/meshes/GRIPPER_L1_1.stl scale=0.001 0.001 0.001
- link GRIPPER_L2_1: geometry collision mesh filename=package://JETANK_description/meshes/GRIPPER_L2_1.stl scale=0.001 0.001 0.001; visual mesh filename=package://JETANK_description/meshes/GRIPPER_L2_1.stl scale=0.001 0.001 0.001
- link GRIPPER_R1_1: geometry collision mesh filename=package://JETANK_description/meshes/GRIPPER_R1_1.stl scale=0.001 0.001 0.001; visual mesh filename=package://JETANK_description/meshes/GRIPPER_R1_1.stl scale=0.001 0.001 0.001
- link GRIPPER_R2_1: geometry collision mesh filename=package://JETANK_description/meshes/GRIPPER_R2_1.stl scale=0.001 0.001 0.001; visual mesh filename=package://JETANK_description/meshes/GRIPPER_R2_1.stl scale=0.001 0.001 0.001
- link SERVO_LOWER_1: geometry collision mesh filename=package://JETANK_description/meshes/SERVO_LOWER_1.stl scale=0.001 0.001 0.001; visual mesh filename=package://JETANK_description/meshes/SERVO_LOWER_1.stl scale=0.001 0.001 0.001
- link SERVO_UPPER_1: geometry collision mesh filename=package://JETANK_description/meshes/SERVO_UPPER_1.stl scale=0.001 0.001 0.001; visual mesh filename=package://JETANK_description/meshes/SERVO_UPPER_1.stl scale=0.001 0.001 0.001
- link base_link: geometry collision mesh filename=package://JETANK_description/meshes/base_link.stl scale=0.001 0.001 0.001; visual mesh filename=package://JETANK_description/meshes/base_link.stl scale=0.001 0.001 0.001

File: JETANK_description/urdf/JETANK.xacro (robot description, xacro)
@@ -568,3 +568,18 @@
   <child link="camera_optical_frame"/>
 </joint>
+<!-- Sensor frame offset 20mm forward (-X in CAMERA_1) to clear the camera housing mesh
+     for the depth camera. The CAMERA_1 mesh extends 14.6mm in -X from the link origin,
+     so 20mm clears it with margin. -->
+<link name="CAMERA_SENSOR_FRAME">
+  <inertial>
+    <origin xyz="0 0 0" rpy="0 0 0"/>
+    <mass value="0.001"/>
+    <inertia ixx="1e-09" iyy="1e-09" izz="1e-09" ixy="0" iyz="0" ixz="0"/>
+  </inertial>
+</link>
+<joint name="camera_sensor_offset_joint" type="fixed">
+  <origin xyz="-0.02 0 0" rpy="0 0 0"/>
+  <parent link="CAMERA_1"/>
+  <child link="CAMERA_SENSOR_FRAME"/>
+</joint>
 </robot>

Commit message: Regenerate JETANK.urdf with cylinder wheel collisions
The merged xacro (origin 02e642f) carries the 4 wheel cylinder collisions +
normalized drive-wheel axes (0 1 0) + continuous wheels + drift-fix dynamics,
but the committed JETANK.urdf was stale (mesh collisions, 0 cylinders) — never
regenerated on either side, which is why the USD built from it had non-rolling
faceted wheels that tipped under drive.

Regenerated from JETANK_description/urdf/JETANK.xacro (ros2 run xacro). Now:
grep -c '<cylinder' == 4 (FREE r=0.02486 l=0.04476, DRIVER r=0.02734 l=0.03903);
both Revolute_DRIVING_WHEEL_R/L axis = (0 1 0); wheels continuous. Mesh paths
normalized file://$(find) -> package:// for portability.

File: JETANK_description/urdf/JETANK.urdf (robot description, URDF)
Before this commit: robot JETANK, 21 links, 20 joints
Links:
- added link CAMERA_SENSOR_FRAME, mass 0.001
- added link base_footprint
- added link camera_optical_frame, mass 0.001
- link DRIVER_WHEEL_L_1: geometry collision cylinder length=0.03903 radius=0.02734; visual mesh filename=package://JETANK_description/meshes/DRIVER_WHEEL_L_1.stl scale=0.001 0.001 0.001
- link DRIVER_WHEEL_R_2: geometry collision cylinder length=0.03903 radius=0.02734; visual mesh filename=package://JETANK_description/meshes/DRIVER_WHEEL_L_1.stl scale=0.001 -0.001 0.001
- link FREE_WHEEL_L_1: geometry collision cylinder length=0.04476 radius=0.02486; visual mesh filename=package://JETANK_description/meshes/FREE_WHEEL_L_1.stl scale=0.001 0.001 0.001
- link FREE_WHEEL_R_1: geometry collision cylinder length=0.04476 radius=0.02486; visual mesh filename=package://JETANK_description/meshes/FREE_WHEEL_L_1.stl scale=0.001 -0.001 0.001
Joints:
- added joint base_joint: type fixed, parent base_footprint, child base_link, origin xyz=0 0 0.08 rpy=0 0 0
- added joint camera_optical_joint: type fixed, parent CAMERA_1, child camera_optical_frame, origin xyz=0 0 0 rpy=-1.5707963 0 -1.5707963
- added joint camera_sensor_offset_joint: type fixed, parent CAMERA_1, child CAMERA_SENSOR_FRAME, origin xyz=-0.02 0 0 rpy=0 0 0
- joint Revolute_DRIVING_WHEEL_L: axis 0.003633 0.999991 0.002097 -> 0 1 0; limit lower=0.0 upper=6.283185 effort=100 velocity=100 -> effort=100 velocity=100; origin xyz=-0.064189 -0.054537 -0.052234 rpy=0 0 0 -> xyz=-0.060 -0.043 -0.051 rpy=0 0 0; type revolute -> continuous
- joint Revolute_DRIVING_WHEEL_R: axis -0.003633 -0.999991 -0.002097 -> 0 1 0; limit lower=0.0 upper=6.283185 effort=100 velocity=100 -> effort=100 velocity=100; origin xyz=0.054631 0.033431 -0.052049 rpy=0 0 0 -> xyz=-0.060 0.043 -0.051 rpy=0 0 0; type revolute -> continuous
- joint Revolute_GRIPPER_R1: limit lower=0.0 upper=1.047198 effort=100 velocity=100 -> lower=0.0 upper=1.047198 effort=1.0 velocity=6.5
- joint Revolute_GRIPPER_R2: limit lower=-1.047198 upper=0.0 effort=100 velocity=100 -> lower=-1.047198 upper=0.0 effort=1.0 velocity=6.5
- joint Revolute_SERVO_LOWER: limit lower=-1.892348 upper=1.574492 effort=100 velocity=100 -> lower=-1.892348 upper=1.574492 effort=2.0 velocity=6.5
- joint Revolute_SERVO_UPPER: limit lower=-1.548620 upper=1.0 effort=100 velocity=100 -> lower=-1.548620 upper=1.0 effort=2.0 velocity=6.5
- joint revolute_BEARING: limit lower=-1.8 upper=1.8 effort=100 velocity=100 -> lower=-1.8 upper=1.8 effort=2.0 velocity=6.5
- joint revolute_CAMERA_HOLDER_ARM_LOWER: limit lower=-1.0 upper=1.0 effort=100 velocity=100 -> lower=-1.0 upper=1.0 effort=2.0 velocity=6.5
- joint revolute_FREE_WHEEL_LEFT: axis 0.003633 0.999991 0.002097 -> 0 1 0; limit lower=0.0 upper=6.283185 effort=100 velocity=100 -> (none); origin xyz=0.05431 -0.054968 -0.052234 rpy=0 0 0 -> xyz=0.054 -0.043 -0.053 rpy=0 0 0; type revolute -> continuous
- joint revolute_FREE_WHEEL_RIGHT: axis -0.003633 -0.999991 -0.002097 -> 0 -1 0; limit lower=0.0 upper=6.283185 effort=100 velocity=100 -> (none); origin xyz=-0.063868 0.033862 -0.052048 rpy=0 0 0 -> xyz=0.054 0.043 -0.053 rpy=0 0 0; type revolute -> continuous
- joint revolute_GRIPPER_L1: limit lower=-1.047198 upper=0.0 effort=100 velocity=100 -> lower=-1.047198 upper=0.0 effort=1.0 velocity=6.5
- joint revolute_GRIPPER_L2: limit lower=-1.047198 upper=0.0 effort=100 velocity=100 -> lower=-1.047198 upper=0.0 effort=1.0 velocity=6.5
